File: rev1.1/split_steno_rev1.1.sch (KiCad schematic (older format))
At the start: 0 parts

Commit message: schematic using keyboard_parts library
Parts:
- added C1: 100, symbol C
- added D1, D10, D11, D12, D13, D14, D15, D16, D17, D18, D2, D3, D4, D5, D6, D7, D8, D9: D, Keebio-Parts:Diode-dual, symbol D
- added D19, D20, D21, D22, D23, D24, D25, D26, D27, D28, D29, D30, D31, D32, D33, D34, D35, D36, D37, D38: LED, symbol LED
- added D?: D, symbol D
- added J1: i2c, Keebio-Parts:TRRS-PJ-320A, symbol Audio-Jack-4
- added J2: rgb, Pin_Headers:Pin_Header_Straight_1x03_Pitch2.54mm, symbol Conn_01x03
- added J3: icsp, Pin_Headers:Pin_Header_Straight_2x03_Pitch2.54mm, symbol Conn_02x03_Odd_Even
- added J4: raw, Pin_Headers:Pin_Header_Straight_1x02_Pitch2.54mm, symbol Conn_01x02
- added J5: serial, Pin_Headers:Pin_Header_Straight_1x04_Pitch2.54mm, symbol Conn_01x04
- added J6: extra, Pin_Headers:Pin_Header_Straight_1x01_Pitch2.54mm, symbol Conn_01x01
- added K1, K10, K11, K12, K13, K14, K15, K16, K17, K18, K19, K2, K20, K3, K4, K5, K6, K7, K8, K9: KEYSW, symbol KEYSW
- added MX?: MX-1U, symbol MX-1U
- added Q1: BC547, symbol BC547
- added R1, R2: 4.7k, symbol R
- added R10, R11, R12, R13, R14, R15, R16, R17, R18, R19, R20, R21, R4, R5, R6, R7, R8, R9: 51, symbol R
- added R22: 1k, symbol R
- added R3: 470, symbol R
- added SW1: reset, Keebio-Parts:SW_Tactile_SPST_Angled_MJTP1117, symbol SW_Push
- added U1: ProMicro, Keebio-Parts:ArduinoProMicro, symbol ProMicro
Connections:
- new net: D1.2, K1.2
- new net: D2.2, K2.2
- new net: D3.2, K3.2
- new net: D4.2, K4.2
- new net: D5.2, K5.2
- new net: D6.2, K6.2
- new net: D7.2, K7.2
- new net: D8.2, K8.2
- new net: D9.2, K9.2
- new net: D10.2, K10.2
- new net: D11.2, K11.2
- new net: D12.2, K12.2
- new net: D13.2, K13.2
- new net: D14.2, K14.2
- new net: D15.2, K15.2
- new net: D16.2, K16.2
- new net: D17.2, K17.2, K19.2
- new net: D18.2, K18.2, K20.2
- new net: D?.2, MX?.2 (ROW)
- new net: J2.2 (Pin_2), R3.1
- new net: D19.1 (K), R4.1
- new net: Q1.1 (C), R10.2, R11.2, R12.2, R13.2, R14.2, R15.2, R16.2, R17.2, R18.2, R19.2, R20.2, R21.2, R4.2, R5.2, R6.2, R7.2, R8.2, R9.2
- new net: Q1.2 (B), R22.1
- new net: D20.1 (K), R5.1
- new net: D21.1 (K), R6.1
- new net: D22.1 (K), R7.1
- new net: D23.1 (K), R8.1
- new net: D24.1 (K), R9.1
- new net: D25.1 (K), R10.1
- new net: D26.1 (K), R11.1
- new net: D27.1 (K), R12.1
- new net: D28.1 (K), R13.1
- new net: D29.1 (K), R14.1
- new net: D30.1 (K), R15.1
- new net: D31.1 (K), R16.1
- new net: D32.1 (K), R17.1
- new net: D33.1 (K), R18.1
- new net: D34.1 (K), R19.1
- new net: D35.1 (K), D36.1 (K), R20.1
- new net: D37.1 (K), D38.1 (K), R21.1
- new net +6V: J4.1 (Pin_1), U1.24 (RAW)
- new net GND: C1.2, J1.4, J2.3 (Pin_3), J3.6 (Pin_6), J4.2 (Pin_2), J5.4 (Pin_4), Q1.3 (E), SW1.2, U1.23 (GND), U1.3 (GND), U1.4 (GND)
- new net VCC: C1.1, D19.2 (A), D20.2 (A), D21.2 (A), D22.2 (A), D23.2 (A), D24.2 (A), D25.2 (A), D26.2 (A), D27.2 (A), D28.2 (A), D29.2 (A), D30.2 (A), D31.2 (A), D32.2 (A), D33.2 (A), D34.2 (A), D35.2 (A), D36.2 (A), D37.2 (A), D38.2 (A), J1.1, J2.1 (Pin_1), J3.2 (Pin_2), J5.1 (Pin_1), R1.2, R2.2, U1.21 (VCC)
- new net c1: K1.1, K11.1, K6.1, U1.19 (F5)
- new net c2: K12.1, K2.1, K7.1, U1.20 (F4)
- new net c3: K13.1, K16.1, K3.1, K8.1, U1.7 (D4)
- new net c4: K14.1, K17.1, K19.1, K4.1, K9.1, U1.8 (C6)
- new net c5: K10.1, K15.1, K18.1, K20.1, K5.1, U1.9 (D7)
- new net d1: J1.2, R1.1, U1.5 (SDA)
- new net d2: J1.3, R2.1, U1.6 (SCL)
- new net d3: R3.2, U1.12 (B5)
- new net d4: J6.1 (Pin_1), R22.2, U1.13 (B6)
- new net miso: J3.1 (Pin_1), U1.15 (B3)
- new net mosi: J3.4 (Pin_4), U1.14 (B2)
- new net r1: D1.1, D2.1, D3.1, D4.1, D5.1, U1.18 (F6)
- new net r2: D10.1, D6.1, D7.1, D8.1, D9.1, U1.17 (F7)
- new net r3: D11.1, D12.1, D13.1, D14.1, D15.1, U1.10 (E6)
- new net r4: D16.1, D17.1, D18.1, U1.11 (B4)
- new net rst: J3.5 (Pin_5), SW1.1, U1.22 (RST)
- new net rx: J5.2 (Pin_2), U1.2 (RX)
- new net sclk: J3.3 (Pin_3), U1.16 (B1)
- new net tx: J5.3 (Pin_3), U1.1 (TX)

Commit message: laid out switch footprints
Parts:
- removed D1: D, Keebio-Parts:Diode-dual, symbol D
- removed D19, D20, D21, D22, D23, D24, D25, D26, D27, D28, D29, D30, D31, D32, D33, D34, D35, D36, D37, D38: LED, symbol LED
- removed K1, K10, K11, K12, K13, K14, K15, K16, K17, K18, K19, K2, K20, K3, K4, K5, K6, K7, K8, K9: KEYSW, symbol KEYSW
- removed R19, R20, R21: 51, symbol R
- added MX10, MX11, MX12, MX13, MX14, MX15, MX16, MX18, MX2, MX20, MX3, MX4, MX5, MX6, MX7, MX8, MX9: MX-1U, Keebio-Parts:Hybrid_PCB_100H_Dual_hole-LED, symbol MX-1U
- added MX17, MX19: MX-1U, Keebio-Parts:Hybrid_PCB_200H-dual-LED, symbol MX-1U
- added R2, R3, R4: 51, Keebio-Parts:Resistor-Hybrid, symbol R
- C1: footprint (none) -> Capacitors_THT:CP_Radial_D5.0mm_P2.00mm
- D1: renamed from D?; footprint (none) -> Keebio-Parts:Diode-dual
- MX1: renamed from MX?; footprint (none) -> Keebio-Parts:Hybrid_PCB_100H_Dual_hole-LED
- Q1: footprint (none) -> TO_SOT_Packages_THT:TO-92_Inline_Narrow_Oval
- R1: renamed from R4; footprint (none) -> Keebio-Parts:Resistor-Hybrid
- R10, R11, R12, R13, R14, R15, R16, R17, R18, R5, R6, R7, R8, R9: footprint (none) -> Keebio-Parts:Resistor-Hybrid
- R19: renamed from R3; footprint (none) -> Keebio-Parts:Resistor-Hybrid
- R20: renamed from R22; footprint (none) -> Keebio-Parts:Resistor-Hybrid
- R21: renamed from R1; footprint (none) -> Keebio-Parts:Resistor-Hybrid
- R22: renamed from R2; footprint (none) -> Keebio-Parts:Resistor-Hybrid
- renumbered J5 to J2, J2 to J3, J3 to J4, J4 to J5
Connections:
- net VCC: now also MX1.3 (LED), MX10.3 (LED), MX11.3 (LED), MX12.3 (LED), MX13.3 (LED), MX14.3 (LED), MX15.3 (LED), MX16.3 (LED), MX17.3 (LED), MX18.3 (LED), MX19.3 (LED), MX2.3 (LED), MX20.3 (LED), MX3.3 (LED), MX4.3 (LED), MX5.3 (LED), MX6.3 (LED), MX7.3 (LED), MX8.3 (LED), MX9.3 (LED)
- net c1: now also MX1.1 (COL), MX11.1 (COL), MX6.1 (COL)
- net c2: now also MX12.1 (COL), MX2.1 (COL), MX7.1 (COL)
- net c3: now also MX13.1 (COL), MX16.1 (COL), MX3.1 (COL), MX8.1 (COL)
- net c4: now also MX14.1 (COL), MX17.1 (COL), MX18.1 (COL), MX4.1 (COL), MX9.1 (COL)
- net c5: now also MX10.1 (COL), MX15.1 (COL), MX19.1 (COL), MX20.1 (COL), MX5.1 (COL)
- net r1: now also D1.1
- net at D2.2: now also MX2.2 (ROW)
- net at D3.2: now also MX3.2 (ROW)
- net at D4.2: now also MX4.2 (ROW)
- net at D5.2: now also MX5.2 (ROW)
- net at D6.2: now also MX6.2 (ROW)
- net at D7.2: now also MX7.2 (ROW)
- net at D8.2: now also MX8.2 (ROW)
- net at D9.2: now also MX9.2 (ROW)
- net at D10.2: now also MX10.2 (ROW)
- net at D11.2: now also MX11.2 (ROW)
- net at D12.2: now also MX12.2 (ROW)
- net at D13.2: now also MX13.2 (ROW)
- net at D14.2: now also MX14.2 (ROW)
- net at D15.2: now also MX15.2 (ROW)
- net at D16.2: now also MX16.2 (ROW)
- net at D17.2: now also MX17.2 (ROW), MX18.2 (ROW)
- net at D18.2: now also MX19.2 (ROW), MX20.2 (ROW)
- net at MX1.4 (LEDGND): now also R1.1
- net at Q1.1 (C), R1.2, R10.2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: now also R2.2, R3.2, R4.2
- net at R5.1: now also MX5.4 (LEDGND)
- net at R6.1: now also MX6.4 (LEDGND)
- net at R7.1: now also MX7.4 (LEDGND)
- net at R8.1: now also MX8.4 (LEDGND)
- net at R9.1: now also MX9.4 (LEDGND)
- net at R10.1: now also MX10.4 (LEDGND)
- net at R11.1: now also MX11.4 (LEDGND)
- net at R12.1: now also MX12.4 (LEDGND)
- net at R13.1: now also MX13.4 (LEDGND)
- net at R14.1: now also MX14.4 (LEDGND)
- net at R15.1: now also MX15.4 (LEDGND)
- net at R16.1: now also MX16.4 (LEDGND)
- net at R17.1: now also MX17.4 (LEDGND), MX18.4 (LEDGND)
- net at R18.1: now also MX19.4 (LEDGND), MX20.4 (LEDGND)
- new net: MX2.4 (LEDGND), R2.1
- new net: MX3.4 (LEDGND), R3.1
- new net: MX4.4 (LEDGND), R4.1
Other:
- moved on the sheet: D1, J6, MX1, Q1, R1, R20

Commit message: removed led from rev1.1, moved to rev1.2
Parts:
- removed MX1, MX10, MX11, MX12, MX13, MX14, MX15, MX16, MX18, MX2, MX20, MX3, MX4, MX5, MX6, MX7, MX8, MX9: MX-1U, Keebio-Parts:Hybrid_PCB_100H_Dual_hole-LED, symbol MX-1U
- removed MX17, MX19: MX-1U, Keebio-Parts:Hybrid_PCB_200H-dual-LED, symbol MX-1U
- removed Q1: BC547, TO_SOT_Packages_THT:TO-92_Inline_Narrow_Oval, symbol BC547
- removed R1, R10, R11, R12, R13, R14, R15, R16, R17, R18, R2, R3, R4, R5, R6, R7, R8, R9: 51, Keebio-Parts:Resistor-Hybrid, symbol R
- removed R20: 1k, Keebio-Parts:Resistor-Hybrid, symbol R
- added K1, K11, K12, K13, K18, K2, K3, K5, K6, K7, K8: KEYSW, Keebio-Parts:Hybrid_PCB_100H_Dual_hole, symbol KEYSW
- added K10, K14, K15, K16, K17, K4, K9: KEYSW, Keebio-Parts:Hybrid_PCB_100H_Dual_hole-flip, symbol KEYSW
- added K19, K20: KEYSW, Keebio-Parts:Hybrid_PCB_200H-dual-nosilk, symbol KEYSW
- renumbered R21 to R1, R22 to R2, R19 to R3
Connections:
- net GND: now also SW1.1; no longer SW1.2
- net c1: now also K1.1, K11.1, K6.1
- net c2: now also K12.1, K2.1, K7.1
- net c3: now also K13.1, K16.1, K3.1, K8.1
- net c4: now also K14.1, K17.1, K19.1, K4.1, K9.1
- net c5: now also K10.1, K15.1, K18.1, K20.1, K5.1
- net d3: now also J6.1 (Pin_1); no longer R3.2
- net d4: now also R3.2; no longer J6.1 (Pin_1)
- net rst: now also SW1.2; no longer SW1.1
- net at D1.2: now also K1.2
- net at D2.2: now also K2.2
- net at D3.2: now also K3.2
- net at D4.2: now also K4.2
- net at D5.2: now also K5.2
- net at D6.2: now also K6.2
- net at D7.2: now also K7.2
- net at D8.2: now also K8.2
- net at D9.2: now also K9.2
- net at D10.2: now also K10.2
- net at D11.2: now also K11.2
- net at D12.2: now also K12.2
- net at D13.2: now also K13.2
- net at D14.2: now also K14.2
- net at D15.2: now also K15.2
- net at D16.2: now also K16.2
- net at D17.2: now also K17.2, K19.2
- net at D18.2: now also K18.2, K20.2
Other:
- moved on the sheet: J6

Commit message: generated gerbers and library managed
Parts:
- C1: footprint Capacitors_THT:CP_Radial_D5.0mm_P2.00mm -> lib_fp:CP_Radial_D5.0mm_P2.00mm
- D1, D10, D11, D12, D13, D14, D15, D16, D17, D18, D2, D3, D4, D5, D6, D7, D8, D9: footprint Keebio-Parts:Diode-dual -> lib_fp:Diode-dual
- J1: footprint Keebio-Parts:TRRS-PJ-320A -> lib_fp:TRRS-PJ-320A
- J2: footprint Pin_Headers:Pin_Header_Straight_1x04_Pitch2.54mm -> lib_fp:Pin_Header_Straight_1x04_Pitch2.54mm
- J3: footprint Pin_Headers:Pin_Header_Straight_1x03_Pitch2.54mm -> lib_fp:Pin_Header_Straight_1x03_Pitch2.54mm
- J4: footprint Pin_Headers:Pin_Header_Straight_2x03_Pitch2.54mm -> lib_fp:Pin_Header_Straight_2x03_Pitch2.54mm
- J5: footprint Pin_Headers:Pin_Header_Straight_1x02_Pitch2.54mm -> lib_fp:Pin_Header_Straight_1x02_Pitch2.54mm
- J6: footprint Pin_Headers:Pin_Header_Straight_1x01_Pitch2.54mm -> lib_fp:Pin_Header_Straight_1x01_Pitch2.54mm
- K1, K11, K12, K13, K18, K2, K3, K5, K6, K7, K8: footprint Keebio-Parts:Hybrid_PCB_100H_Dual_hole -> lib_fp:Hybrid_PCB_100H_Dual_hole
- K10, K14, K15, K16, K17, K4, K9: footprint Keebio-Parts:Hybrid_PCB_100H_Dual_hole-flip -> lib_fp:Hybrid_PCB_100H_Dual_hole-flip
- K19, K20: footprint Keebio-Parts:Hybrid_PCB_200H-dual-nosilk -> lib_fp:Hybrid_PCB_200H-dual-nosilk
- R1, R2, R3: footprint Keebio-Parts:Resistor-Hybrid -> lib_fp:Resistor-Hybrid
- SW1: footprint Keebio-Parts:SW_Tactile_SPST_Angled_MJTP1117 -> lib_fp:SW_Tactile_SPST_Angled_MJTP1117
- U1: footprint Keebio-Parts:ArduinoProMicro -> lib_fp:ArduinoProMicro
