File: rev1.1/split_steno_rev1.1.kicad_pcb (KiCad board)
At the start: 2 copper layers, 99.4 x 84.8 mm, 61 parts, among them J1 i2c, J2 serial, J3 rgb, J4 icsp, J5 raw, J6 extra, K1 KEYSW, K10 KEYSW, K11 KEYSW, K12 KEYSW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

Commit message: one last thing
Parts:
- C1: footprint Capacitors_THT:CP_Radial_D5.0mm_P2.00mm -> lib_fp:CP_Radial_D5.0mm_P2.00mm
- D1, D10, D11, D12, D13, D14, D15, D16, D17, D18, D2, D3, D4, D5, D6, D7, D8, D9: footprint Keebio-Parts:Diode-dual -> lib_fp:Diode-dual
- J1: footprint Keebio-Parts:TRRS-PJ-320A -> lib_fp:TRRS-PJ-320A
- J2: footprint Pin_Headers:Pin_Header_Straight_1x04_Pitch2.54mm -> lib_fp:Pin_Header_Straight_1x04_Pitch2.54mm
- J3: footprint Pin_Headers:Pin_Header_Straight_1x03_Pitch2.54mm -> lib_fp:Pin_Header_Straight_1x03_Pitch2.54mm
- J4: footprint Pin_Headers:Pin_Header_Straight_2x03_Pitch2.54mm -> lib_fp:Pin_Header_Straight_2x03_Pitch2.54mm
- J5: footprint Pin_Headers:Pin_Header_Straight_1x02_Pitch2.54mm -> lib_fp:Pin_Header_Straight_1x02_Pitch2.54mm
- J6: footprint Pin_Headers:Pin_Header_Straight_1x01_Pitch2.54mm -> lib_fp:Pin_Header_Straight_1x01_Pitch2.54mm
- K1, K11, K12, K13, K18, K2, K3, K5, K6, K7, K8: footprint Keebio-Parts:Hybrid_PCB_100H_Dual_hole -> lib_fp:Hybrid_PCB_100H_Dual_hole
- K10, K14, K15, K16, K17, K4, K9: footprint Keebio-Parts:Hybrid_PCB_100H_Dual_hole-flip -> lib_fp:Hybrid_PCB_100H_Dual_hole-flip
- K19, K20: footprint Keebio-Parts:Hybrid_PCB_200H-dual-nosilk -> lib_fp:Hybrid_PCB_200H-dual-nosilk
- R1, R2, R3: footprint Keebio-Parts:Resistor-Hybrid -> lib_fp:Resistor-Hybrid
- SW1: footprint Keebio-Parts:SW_Tactile_SPST_Angled_MJTP1117 -> lib_fp:SW_Tactile_SPST_Angled_MJTP1117
- U1: footprint Keebio-Parts:ArduinoProMicro -> lib_fp:ArduinoProMicro
