File: rev2.0/split_steno_rev2.0.kicad_pcb (KiCad board)
At the start: 2 copper layers, 0 parts

Commit message: begin pcb file
Parts:
- added BT1: Battery, Battery_Holders:Keystone_1058_1x2032-CoinCell, B.Cu at (107.2, 102.4)
- added BT2: Battery_Cell, Connectors_JST:JST_PH_S2B-PH-K_02x2.00mm_Angled, B.Cu at (290.0, 175.5)
- added C1: 4.7uF, Capacitors_SMD:C_0603_HandSoldering, B.Cu at (288.8, 157.1)
- added C10: 0.1uF, Capacitors_SMD:C_0603_HandSoldering, B.Cu at (306.6, 171.8)
- added C11: 0.1uF, Capacitors_SMD:C_0603_HandSoldering, B.Cu at (254.0, 121.3)
- added C12: 47uF, Capacitors_SMD:C_0603_HandSoldering, B.Cu at (309.6, 183.4)
- added C13: 0.1uF, Capacitors_SMD:C_0603_HandSoldering, B.Cu at (284.4, 152.1)
- added C14: 10uF, Capacitors_SMD:C_0603_HandSoldering, B.Cu at (256.9, 138.0)
- added C2: 0.1uF, Capacitors_SMD:C_0603_HandSoldering, B.Cu at (273.0, 135.4)
- added C3: 0.1uF, Capacitors_SMD:C_0603_HandSoldering, B.Cu at (284.4, 147.3)
- added C4: 0.1uF, Capacitors_SMD:C_0603_HandSoldering, B.Cu at (288.9, 152.3)
- added C5: 0.1uF, Capacitors_SMD:C_0603_HandSoldering, B.Cu at (254.0, 116.5)
- added C6: 4.7uF, Capacitors_SMD:C_0603_HandSoldering, B.Cu at (258.5, 121.8)
- added C7: 1uF, Capacitors_SMD:C_0603_HandSoldering, B.Cu at (296.6, 158.2)
- added C8: 1uF, Capacitors_SMD:C_0603_HandSoldering, B.Cu at (309.6, 178.6)
- added C9: 0.1uF, Capacitors_SMD:C_0603_HandSoldering, B.Cu at (264.5, 128.8)
- added D1: D_Schottky_x2_KCom_AAK, TO_SOT_Packages_SMD:SOT-23_Handsoldering, B.Cu at (172.1, 154.6)
- added F1: Fuse, Fuse_Holders_and_Fuses:Fuse_SMD1206_HandSoldering, B.Cu at (298.2, 164.0)
- added J1: Audio-Jack-4, Keebio-Parts:TRRS-PJ-320A, F.Cu at (102.4, 52.4)
- added J2: USB_OTG, keyboard_parts:USB_miniB, B.Cu at (69.1, 69.1)
- added JP1: Jumper, keyboard_parts:SOLDER_JUMPER_2, B.Cu at (234.8, 111.3)
- added JP2: Jumper, keyboard_parts:SOLDER_JUMPER_2, B.Cu at (249.9, 126.1)
- added JP3: Jumper, keyboard_parts:SOLDER_JUMPER_2, B.Cu at (230.1, 111.3)
- added LED1: WS2812B, WS2812B:WS2812B, B.Cu at (50.0, 69.1)
- added LED2: WS2812B, WS2812B:WS2812B, B.Cu at (107.2, 69.1)
- added LED3: WS2812B, WS2812B:WS2812B, B.Cu at (50.0, 116.7)
- added LED4: WS2812B, WS2812B:WS2812B, B.Cu at (107.2, 116.7)
- added P1: TC2030-IDC, Connectors:Tag-Connect_TC2030-IDC-NL, B.Cu at (214.1, 112.9)
- added R1: 10k, Resistors_SMD:R_0603_HandSoldering, B.Cu at (239.3, 111.4)
- added R2: 470k, Resistors_SMD:R_0603_HandSoldering, B.Cu at (297.8, 171.5)
- added R3: 470k, Resistors_SMD:R_0603_HandSoldering, B.Cu at (284.3, 156.9)
- added R4: 100k, Resistors_SMD:R_0603_HandSoldering, B.Cu at (297.8, 176.5)
- added R5: 100k, Resistors_SMD:R_0603_HandSoldering, B.Cu at (268.6, 135.2)
- added R6: 10k, Resistors_SMD:R_0603_HandSoldering, B.Cu at (272.9, 140.2)
- added R7: 4.7k, Resistors_SMD:R_0603_HandSoldering, B.Cu at (268.6, 140.2)
- added R8: 100k, Resistors_SMD:R_0603_HandSoldering, B.Cu at (302.2, 171.6)
- added R9: 4.7k, Resistors_SMD:R_0603_HandSoldering, B.Cu at (277.0, 145.6)
- added REF**: TRRS-PJ-320A, Keebio-Parts:TRRS-PJ-320A, B.Cu at (95.2, 52.4)
- added SW1: SW_Push, Keebio-Parts:Hybrid_PCB_100H_Dual_hole, F.Cu at (40.5, 73.8)
- added SW10: SW_Push, Keebio-Parts:Hybrid_PCB_100H_Dual_hole, F.Cu at (116.7, 92.9)
- added SW11: SW_Push, Keebio-Parts:Hybrid_PCB_100H_Dual_hole, F.Cu at (40.5, 111.9)
- added SW12: SW_Push, Keebio-Parts:Hybrid_PCB_100H_Dual_hole, F.Cu at (59.5, 111.9)
- added SW13: SW_Push, Keebio-Parts:Hybrid_PCB_100H_Dual_hole, F.Cu at (78.6, 111.9)
- added SW14: SW_Push, Keebio-Parts:Hybrid_PCB_100H_Dual_hole, F.Cu at (97.6, 111.9)
- added SW15: SW_Push, Keebio-Parts:Hybrid_PCB_100H_Dual_hole, F.Cu at (116.7, 111.9)
- added SW16: SW_Push, Keebio-Parts:Hybrid_PCB_100H_Dual_hole, F.Cu at (88.1, 131.0)
- added SW17: SW_Push, Keebio-Parts:Hybrid_PCB_100H_Dual_hole, F.Cu at (107.2, 131.0)
- added SW18: SW_Push, Keebio-Parts:Hybrid_PCB_100H_Dual_hole, F.Cu at (126.2, 131.0)
- added SW19: SW_Push, Keebio-Parts:Hybrid_PCB_200H-dual-nosilk, F.Cu at (97.6, 131.0)
- added SW2: SW_Push, Keebio-Parts:Hybrid_PCB_100H_Dual_hole, F.Cu at (59.5, 73.8)
- added SW20: SW_Push, Keebio-Parts:Hybrid_PCB_200H-dual-nosilk, F.Cu at (116.7, 131.0)
- added SW21: Switch-6P-2S2T, switch:SlideSwitch_C&K_JS202011CQN, B.Cu at (235.1, 118.4)
- added SW22: SW_Push, switch:SwitchPush_C&K_MultiFoot_RS-187R05A2-DS_And_PTS645_SMT, B.Cu at (154.8, 83.3)
- added SW3: SW_Push, Keebio-Parts:Hybrid_PCB_100H_Dual_hole, F.Cu at (78.6, 73.8)
- added SW4: SW_Push, Keebio-Parts:Hybrid_PCB_100H_Dual_hole, F.Cu at (97.6, 73.8)
- added SW5: SW_Push, Keebio-Parts:Hybrid_PCB_100H_Dual_hole, F.Cu at (116.7, 73.8)
- added SW6: SW_Push, Keebio-Parts:Hybrid_PCB_100H_Dual_hole, F.Cu at (40.5, 92.9)
- added SW7: SW_Push, Keebio-Parts:Hybrid_PCB_100H_Dual_hole, F.Cu at (59.5, 92.9)
- added SW8: SW_Push, Keebio-Parts:Hybrid_PCB_100H_Dual_hole, F.Cu at (78.6, 92.9)
- added SW9: SW_Push, Keebio-Parts:Hybrid_PCB_100H_Dual_hole, F.Cu at (97.6, 92.9)
- added U1: 74LVC1G34, TO_SOT_Packages_SMD:SOT-353_SC-70-5_Handsoldering, B.Cu at (223.3, 113.2)
- added U2: MCP73831, TO_SOT_Packages_SMD:SOT-23-5_HandSoldering, B.Cu at (290.4, 163.3)
- added U3: MCP1700, TO_SOT_Packages_SMD:SOT-23, B.Cu at (185.6, 154.6)
- added U4: MCP1700, TO_SOT_Packages_SMD:SOT-23, B.Cu at (258.6, 127.6)
- added U5: ATXMEGA128A4U-AU, Housings_QFP:TQFP-44_10x10mm_Pitch0.8mm, B.Cu at (69.1, 102.4)
- added U6: nRF24L01_module, nordic:NRF24L01-Module-SMD, B.Cu at (50.0, 102.4)

Commit message: pcb
Parts:
- added LED4: VAL**, WS2812B:WS2812B, F.Cu at (138.1, 114.3)
- added REF**: MountingHole_2.2mm_M2_Pad, Mounting_Holes:MountingHole_2.2mm_M2_Pad, F.Cu at (116.7, 121.4)
- added REF**: MountingHole_2.2mm_M2_Pad, Mounting_Holes:MountingHole_2.2mm_M2_Pad, F.Cu at (40.5, 121.4)
- added REF**: MountingHole_2.2mm_M2_Pad, Mounting_Holes:MountingHole_2.2mm_M2_Pad, F.Cu at (116.7, 64.3)
- added REF**: MountingHole_2.2mm_M2_Pad, Mounting_Holes:MountingHole_2.2mm_M2_Pad, F.Cu at (40.5, 64.3)
- moved R8 269.0 mm to (71.4, 33.3)
- moved F1 265.4 mm to (71.4, 26.2)
- moved R9 179.4 mm to (133.3, 38.1)
- moved R7 174.4 mm to (132.9, 30.7)
- moved R6 121.7 mm to (166.7, 81.0)
- moved C1 57.3 mm to (250.7, 114.2)
- moved C7 57.3 mm to (258.5, 115.3)
- moved C8 57.3 mm to (271.5, 135.8)
- moved C13 57.3 mm to (246.3, 109.2)
- moved C14 57.3 mm to (218.8, 95.2)
- moved C3 57.3 mm to (246.3, 104.4)
- moved C6 57.3 mm to (220.4, 78.9)
- moved SW21 57.3 mm to (197.0, 75.5)
- moved U1 57.3 mm to (185.2, 70.4)
- moved U2 57.3 mm to (252.3, 120.4)
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