File: rev3.0/split_steno_right.kicad_pcb (KiCad board)
At the start: 2 copper layers, 99.7 x 74.2 mm, 44 parts, among them J1 USB_B, J2 Audio-Jack-4, J3 Conn_02x04_Odd_Even, J4 Conn_01x03, J5 Conn_01x03, J6 Conn_01x02, M2 MountingHole_2.2mm_M2, P1 TC2030-IDC, SW1 SW_Push, SW10 SW_Push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

Commit message: finished right hand
Parts:
- removed J6: Conn_01x02, lib_fp:Pin_Header_Straight_1x02_Pitch2.54mm
- added G***: LOGO, lib_fp:airi_icon-7.6, B.Cu at (81.0, 80.5)
- G***: footprint airi_logo:airi_icon-7.6 -> lib_fp:airi_icon-7.6
- J4: value Conn_01x03 -> Conn_01x02; footprint lib_fp:Pin_Header_Straight_1x03_Pitch2.54mm -> lib_fp:Pin_Header_Straight_1x02_Pitch2.54mm
- J5: value Conn_01x03 -> Conn_02x04_Odd_Even; footprint lib_fp:Pin_Header_Straight_1x03_Pitch2.54mm -> lib_fp:Pin_Header_Straight_2x04_Pitch2.54mm
- M2 (x6): footprint Mounting_Holes:MountingHole_2.2mm_M2 -> lib_fp:MountingHole_2.2mm_M2
- moved J5 52.8 mm to (139.3, 75.7), turned to 180 degrees
- moved J4 18.4 mm to (119.9, 77.2), turned to 270 degrees
- moved C2 0.10 mm to (117.5, 80.3)
Connections:
- J1 pad 6: (no net) -> GND
- J4 pad 1: VCC -> /EXTRA1
- J4 pad 2: Net-(J4-Pad2) -> GND
- J5 pad 1: VCC -> GND
- J5 pad 2: Net-(J5-Pad2) -> VCC
- J5 pad 3: GND -> /EXTRA3
- U2 pad 1: Net-(U2-Pad1) -> /KEY11
- U2 pad 2: Net-(U2-Pad2) -> /KEY6
- U2 pad 20: Net-(U2-Pad20) -> /KEY8
- U2 pad 21: Net-(U2-Pad21) -> /KEY10
- U2 pad 22: Net-(U2-Pad22) -> /KEY5
- U2 pad 23: Net-(U2-Pad23) -> /KEY9
- U2 pad 24: Net-(U2-Pad24) -> /KEY4
- U2 pad 25: Net-(U2-Pad25) -> /KEY3
- U2 pad 3: Net-(U2-Pad3) -> /KEY12
- U2 pad 32: Net-(U2-Pad32) -> /KEY7
- U2 pad 37: Net-(U2-Pad37) -> /EXTRA1
- U2 pad 4: Net-(U2-Pad4) -> /KEY16
- U2 pad 40: Net-(U2-Pad40) -> /EXTRA2
- U2 pad 41: Net-(U2-Pad41) -> /EXTRA3
- U2 pad 42: Net-(U2-Pad42) -> /EXTRA4
- U2 pad 43: Net-(U2-Pad43) -> /EXTRA5
- U2 pad 44: Net-(U2-Pad44) -> /EXTRA6
- U2 pad 5: Net-(U2-Pad5) -> /KEY17
- U2 pad 6: Net-(U2-Pad6) -> /KEY13
- U2 pad 7: Net-(U2-Pad7) -> /KEY18
Routing:
- net Net-(U2-Pad42): track 68.5 -> 0.00 mm
- net /KEY10: track 0.00 -> 65.6 mm
- net /KEY5: track 0.00 -> 65.3 mm
- net Net-(U2-Pad43): track 58.9 -> 0.00 mm
- net GND: track 129.7 -> 72.6 mm
- net VCC: track 153.8 -> 206.6 mm
- net Net-(U2-Pad44): track 52.4 -> 0.00 mm
- net /KEY6: track 0.00 -> 50.2 mm
- net /KEY4: track 9.19 -> 43.4 mm
- net Net-(U2-Pad24): track 34.2 -> 0.00 mm
- net Net-(U2-Pad22): track 33.4 -> 0.00 mm
- net /KEY17: track 53.0 -> 85.7 mm
- net Net-(U2-Pad4): track 29.8 -> 0.00 mm
- net /EXTRA3: track 0.00 -> 28.9 mm
- net /KEY16: track 31.4 -> 59.5 mm
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Other:
- board text removed: "jtallbean"
